Commit message: backup namespace change version

File: src/pinklab_minibot_robot/minibot_description/urdf/minibot.urdf.xacro (robot description, xacro)
@@ -2,6 +2,8 @@
 <robot xmlns:xacro="http://www.ros.org/wiki/xacro">
     <xacro:macro name="insert_robot" params="prefix">
+        <xacro:arg name="namespace" default="robot1/"/>
         <xacro:property name="wheel_diameter" value="0.068"/>
         <xacro:property name="wheel_speration" value="0.180"/>
+        <xacro:property name="prefix" value="$(arg namespace)"/>
         <link name="${prefix}base_footprint"/>
         <link name="${prefix}base_link">

File: src/pinklab_minibot_robot/minibot_description/urdf/robot.urdf.xacro (robot description, xacro)
@@ -5,9 +5,12 @@
     <xacro:include filename="$(find minibot_description)/urdf/minibot_gazebo.urdf.xacro"/>
     <xacro:include filename="$(find minibot_description)/urdf/minibot_ros2_control.urdf.xacro"/>
+    <xacro:arg name="namespace" default="robot1/"/>
     <xacro:arg name="prefix" default=""/>
+    <!-- <xacro:arg name="prefix" default="$(arg namespace)"/> -->
     <xacro:arg name="is_sim" default="false"/>
     <xacro:arg name="robot_port_name" default="/dev/ttyArduino"/>
     <xacro:arg name="robot_baudrate" default="500000"/>
     <xacro:property name="prefix" value="$(arg prefix)"/>
+    <!-- <xacro:property name="prefix" value="$(arg namespace)"/> -->
     <!-- insert robot base -->
     <xacro:insert_robot prefix="$(arg prefix)"/>
